Commit message: Updated robot_control

File: src/trace_description/description/robot.urdf.xacro (robot description, xacro)
@@ -2,5 +2,6 @@
 <robot xmlns:xacro="http://www.ros.org/wiki/xacro"  name="robot">
     <xacro:arg name="use_ros2_control" default="true"/>
-    <xacro:include filename="robot_core.xacro" />
+    <xacro:include filename="trace_core.xacro" />
+    <xacro:include filename = "depth_camera.xacro"/>
     <!-- Switch between ros2_control and Gazebo integrated diff-drive control -->
     <xacro:if value="$(arg use_ros2_control)">
@@ -10,7 +11,6 @@
         <xacro:include filename="gazebo_control.xacro" />
     </xacro:unless>
-    <!--<xacro:include filename = "gazebo_control.xacro"/>-->
     <!-- <xacro:include filename = "lidar.xacro"/>  Deactivating Lidar for now because I do not need it-->
     <!--<xacro:include filename = "camera.xacro"/>-->
-    <xacro:include filename = "depth_camera.xacro"/>
+    <!--<xacro:include filename="robot_core.xacro" />-->
 </robot>

File: src/trace_description/description/ros2_control.xacro (robot description, xacro)
@@ -1,5 +1,28 @@
 <?xml version="1.0"?>
 <robot xmlns:xacro="http://www.ros.org/wiki/xacro">
-    <ros2_control name="GazeboSystem" type = "system">
+        <ros2_control name="RealRobot" type="system">
+            <hardware>
+                <plugin>trace_firmware/TraceInterface</plugin>
+                <param name="port">/dev/ttyDC</param>
+            </hardware>
+            <!-- Note everything below here is the same as the Gazebo one -->
+            <joint name="left_wheel_joint">
+                <command_interface name="velocity">
+                    <param name="min">-10</param>
+                    <param name="max">10</param>
+                </command_interface>
+                <state_interface name="position"/>
+                <state_interface name="velocity"/>
+            </joint>
+            <joint name="right_wheel_joint">
+                <command_interface name="velocity">
+                    <param name="min">-10</param>
+                    <param name="max">10</param>
+                </command_interface>
+                <state_interface name="position"/>
+                <state_interface name="velocity"/>
+            </joint>
+        </ros2_control>
+    <!--<ros2_control name="GazeboSystem" type = "system">
         <hardware>
             <plugin>gz_ros2_control/GazeboSimSystem</plugin>
@@ -21,5 +44,5 @@
             <state_interface name = "position"/>
         </joint>
-    </ros2_control>
+    </ros2_control>-->
     <gazebo>
         <plugin name="gz_ros2_control::GazeboSimROS2ControlPlugin" filename="libgz_ros2_control-system.so">
