Commit message: added ball_collect_node

File: src/trace_description/description/camera.xacro (robot description, xacro)
@@ -5,21 +5,90 @@
             <parent link = "chassis_link"/>
             <child link = "camera_link"/>
-            <origin xyz = "0.305 0 0.08" rpy = "0 0 0"/>
+            <origin xyz = "0 0 0" rpy = "0 0 0"/>
         </joint>
-        <link name = "camera_link">
+        <joint name="base_camera_joint" type="fixed">
+            <origin xyz="${xyz}" rpy="${rpy}" />
+            <parent link="${parent_frame}" />
+            <origin xyz="0 0 0" rpy="0 0 0" />
+            <child link="camera_link" />
+        </joint>
+        <link name="camera_link">
+            <inertial>
+            <mass value="0.01" />
+            <origin xyz="0 0 0" />
+            <inertia ixx="0.001" ixy="0.0" ixz="0.0"
+                iyy="0.001" iyz="0.0"
+                izz="0.001" />
+            </inertial>
             <visual>
-                <geometry>
-                    <box size = "0.010 0.03 0.03"/>
-                </geometry>
+            <origin xyz=" 0 0 0 " rpy="0 0 0" />
+            <geometry>
+                <mesh filename="package://kinect_description/meshes/kinect.dae"/>
+            </geometry>
             </visual>
+            <collision>
+            <origin xyz="0.0 0.0 0.0" rpy="0 0 0" />
+            <geometry>
+                <box size="0.0730 .2760 0.0720"/>
+            </geometry>
+            </collision>
         </link>
-        <joint name = "camera_optical_joint" type = "fixed">
-            <parent link = "camera_link"/>
-            <child link = "camera_link_optical"/>
-            <origin xyz = "0 0 0" rpy = "${-pi/2} 0 ${-pi/2} "/>
+        <joint name="camera_depth_joint" type="fixed">
+            <origin xyz="0 0.011 0" rpy="0 0 0" />
+            <parent link="camera_link" />
+            <child link="camera_depth_frame" />
         </joint>
-        <link name = "camera_link_optical">
+        <link name="camera_depth_frame">
+            <inertial>
+            <mass value="0.01" />
+            <origin xyz="0 0 0" />
+            <inertia ixx="0.001" ixy="0.0" ixz="0.0"
+                iyy="0.001" iyz="0.0"
+                izz="0.001" />
+            </inertial>
         </link>
-    <gazebo reference="camera_link">
+        <joint name="camera_depth_optical_joint" type="fixed">
+            <origin xyz="0 0 0" rpy="${-M_PI/2} 0 ${-M_PI/2}" />
+            <parent link="camera_depth_frame" />
+            <child link="camera_depth_optical_frame" />
+        </joint>
+        <link name="camera_depth_optical_frame">
+            <inertial>
+            <mass value="0.001" />
+            <origin xyz="0 0 0" />
+            <inertia ixx="0.0001" ixy="0.0" ixz="0.0"
+                iyy="0.0001" iyz="0.0"
+                izz="0.0001" />
+            </inertial>
+        </link>
+        <joint name="camera_rgb_joint" type="fixed">
+            <origin xyz="0 -0.012 0" rpy="0 0 0" />
+            <parent link="camera_link" />
+            <child link="camera_rgb_frame" />
+        </joint>
+        <link name="camera_rgb_frame">
+            <inertial>
+            <mass value="0.001" />
+            <origin xyz="0 0 0" />
+            <inertia ixx="0.0001" ixy="0.0" ixz="0.0"
+                iyy="0.0001" iyz="0.0"
+                izz="0.0001" />
+            </inertial>
+        </link>
+        <joint name="camera_rgb_optical_joint" type="fixed">
+            <origin xyz="0 0 0" rpy="${-M_PI/2} 0 ${-M_PI/2}" />
+            <parent link="camera_rgb_frame" />
+            <child link="camera_rgb_optical_frame" />
+        </joint>
+        <link name="camera_rgb_optical_frame">
+            <inertial>
+            <mass value="0.001" />
+            <origin xyz="0 0 0" />
+            <inertia ixx="0.0001" ixy="0.0" ixz="0.0"
+                iyy="0.0001" iyz="0.0"
+                izz="0.0001" />
+            </inertial>
+        </link>
+    <!--<gazebo reference="camera_link">
         <sensor name="camera" type="camera">
             <pose> 0 0 0 0 0 0 </pose>
@@ -42,4 +111,4 @@
             <gz_frame_id>camera_link_optical</gz_frame_id>
         </sensor>
-    </gazebo>
+    </gazebo>-->
 </robot>

File: src/trace_description/description/depth_camera.xacro (robot description, xacro)
@@ -2,24 +2,87 @@
 <robot xmlns:xacro="http://www.ros.org/wiki/xacro">
     <xacro:property name="mesh_path" value="file://$(find trace_description)/meshes"/>
-        <joint name = "camera_joint" type="fixed">
-            <parent link = "chassis_link"/>
-            <child link = "camera_link"/>
-            <origin xyz = "0.305 0 0.08" rpy = "0 0 0"/>
-        </joint>
-        <link name = "camera_link">
-            <visual>
-                <geometry>
-                    <box size = "0.010 0.03 0.03"/>
-                </geometry>
-            </visual>
-        </link>
-        <joint name = "camera_optical_joint" type = "fixed">
-            <parent link = "camera_link"/>
-            <child link = "camera_link_optical"/>
-            <origin xyz = "0 0 0" rpy = "${-pi/2} 0 ${-pi/2} "/>
-        </joint>
-        <link name = "camera_link_optical">
-        </link>
-    <gazebo reference="camera_link">
+    <joint name = "camera_joint" type="fixed">
+        <parent link = "chassis_link"/>
+        <child link = "camera_link"/>
+        <origin xyz = "0.14 0 0.28" rpy = "0 0 0"/>
+    </joint>
+  <link name="camera_link">
+    <inertial>
+        <mass value="0.01" />
+        <origin xyz="0 0 0" />
+        <inertia ixx="0.001" ixy="0.0" ixz="0.0"
+            iyy="0.001" iyz="0.0"
+            izz="0.001" />
+    </inertial>
+    <visual>
+        <origin xyz=" 0 0 0 " rpy="0 0 0" />
+        <geometry>
+            <mesh filename="package://trace_description/meshes/kinect.dae"/>
+        </geometry>
+    </visual>
+    <collision>
+        <origin xyz="0.0 0.0 0.0" rpy="0 0 0" />
+        <geometry>
+            <box size="0.0730 .2760 0.0720"/>
+        </geometry>
+    </collision>
+  </link>
+  <joint name="camera_depth_joint" type="fixed">
+    <origin xyz="0 0.011 0" rpy="0 0 0" />
+    <parent link="camera_link" />
+    <child link="camera_depth_frame" />
+  </joint>
+  <link name="camera_depth_frame">
+    <inertial>
+      <mass value="0.01" />
+      <origin xyz="0 0 0" />
+      <inertia ixx="0.001" ixy="0.0" ixz="0.0"
+        iyy="0.001" iyz="0.0"
+        izz="0.001" />
+    </inertial>
+  </link>
+  <joint name="camera_depth_optical_joint" type="fixed">
+    <origin xyz="0 0 0" rpy="${-pi/2} 0 ${-pi/2}" />
+    <parent link="camera_depth_frame" />
+    <child link="camera_depth_optical_frame" />
+  </joint>
+  <link name="camera_depth_optical_frame">
+    <inertial>
+      <mass value="0.001" />
+      <origin xyz="0 0 0" />
+      <inertia ixx="0.0001" ixy="0.0" ixz="0.0"
+        iyy="0.0001" iyz="0.0"
+        izz="0.0001" />
+    </inertial>
+  </link>
+  <joint name="camera_rgb_joint" type="fixed">
+    <origin xyz="0 -0.012 0" rpy="0 0 0" />
+    <parent link="camera_link" />
+    <child link="camera_rgb_frame" />
+  </joint>
+  <link name="camera_rgb_frame">
+    <inertial>
+      <mass value="0.001" />
+      <origin xyz="0 0 0" />
+      <inertia ixx="0.0001" ixy="0.0" ixz="0.0"
+        iyy="0.0001" iyz="0.0"
+        izz="0.0001" />
+    </inertial>
+  </link>
+  <joint name="camera_rgb_optical_joint" type="fixed">
+    <origin xyz="0 0 0" rpy="${-pi/2} 0 ${-pi/2}" />
+    <parent link="camera_rgb_frame" />
+    <child link="camera_rgb_optical_frame" />
+  </joint>
+  <link name="camera_rgb_optical_frame">
+    <inertial>
+      <mass value="0.001" />
+      <origin xyz="0 0 0" />
+      <inertia ixx="0.0001" ixy="0.0" ixz="0.0"
+        iyy="0.0001" iyz="0.0"
+        izz="0.0001" />
+    </inertial>
+  </link>
+    <!--<gazebo reference="camera_link">
         <sensor name="rgbd_camera" type="rgbd_camera">
             <camera>
@@ -41,4 +104,4 @@
             <gz_frame_id>camera_link</gz_frame_id>
         </sensor>
-  </gazebo>
+  </gazebo>-->
 </robot>

File: src/trace_description/description/ros2_control.xacro (robot description, xacro)
@@ -24,25 +24,27 @@
             </joint>
         </ros2_control>
-    <!--<ros2_control name="GazeboSystem" type = "system">
-        <hardware>
-            <plugin>gz_ros2_control/GazeboSimSystem</plugin>
-        </hardware>
-        <joint name = "left_wheel_joint">
-            <command_interface name = "velocity">
-                <param name = "min">-10</param>
-                <param name = "max">10</param>
-            </command_interface>
-            <state_interface name = "velocity"/>
-            <state_interface name = "position"/>
-        </joint>
-        <joint name = "right_wheel_joint">
-            <command_interface name = "velocity">
-                <param name = "min">-10</param>
-                <param name = "max">10</param>
-            </command_interface>
-            <state_interface name = "velocity"/>
-            <state_interface name = "position"/>
-        </joint>
-    </ros2_control>-->
+    <!--<xacro:if value="$(arg use_sim_mode)">
+        <ros2_control name="GazeboSystem" type="system">
+            <hardware>
+                <plugin>gazebo_ros2_control/GazeboSystem</plugin>
+            </hardware>
+            <joint name="left_wheel_joint">
+                <command_interface name="velocity">
+                    <param name="min">-10</param>
+                    <param name="max">10</param>
+                </command_interface>
+                <state_interface name="velocity"/>
+                <state_interface name="position"/>
+            </joint>
+            <joint name="right_wheel_joint">
+                <command_interface name="velocity">
+                    <param name="min">-10</param>
+                    <param name="max">10</param>
+                </command_interface>
+                <state_interface name="velocity"/>
+                <state_interface name="position"/>
+            </joint>
+        </ros2_control>
+    </xacro:if>-->
     <gazebo>
         <plugin name="gz_ros2_control::GazeboSimROS2ControlPlugin" filename="libgz_ros2_control-system.so">

File: src/trace_description/description/trace_core.xacro (robot description, xacro)
@@ -27,5 +27,5 @@
         <parent link = "base_link"/>
         <child link = "chassis_link"/>
-        <origin xyz = "-0.1 0 0"/> <!-- We want the chassis link to sit at the edge of the chassis (100 cm behind the wheels)-->
+        <origin xyz = "-0.345 0 0.035"/> <!-- We want the chassis link to sit at the edge of the chassis (100 cm behind the wheels)-->
     </joint>
     <!-- By default the visual of the link centers around the location of the joint
@@ -33,18 +33,19 @@
     <link name = "chassis_link">
         <visual>
-            <origin xyz = "0.15 0 0.075"/>
+            <origin xyz = "0.26 -0.130 0.170"/>
             <geometry>
-                <box size = "0.3 0.3 0.15"/>
+                <!--<box size = "0.520 0.410 0.055"/>-->
+                <mesh filename="package://trace_description/meshes/chassis.stl" />
             </geometry>
             <material name = "white"/>
         </visual>
         <collision>
-            <origin xyz = "0.15 0 0.075"/>
+            <origin xyz = "0.26 0 0.0275"/>
             <geometry>
-                <box size = "0.3 0.3 0.15"/>
+                <box size = "0.520 0.410 0.055"/>
             </geometry>
         </collision>
-        <xacro:inertial_box mass = "0.5" x = "0.3" y = "0.3" z = "0.15">
-            <origin xyz = "0.15 0 0.075" rpy = "0 0 0"/>
+        <xacro:inertial_box mass="2.0" x="0.520" y="0.410" z="0.055">
+            <origin xyz="0.26 0 0.0275" rpy="0 0 0"/>
         </xacro:inertial_box>
     </link>
@@ -55,5 +56,5 @@
         <parent link = "base_link"/>
         <child link = "left_wheel_link"/>
-        <origin xyz = "0 0.175 0" rpy = "-${pi/2} 0 0"/>
+        <origin xyz = "0 0.255 0" rpy = "-${pi/2} 0 0"/>
         <axis xyz = "0 0 1"/>
         <limit effort="0.05" velocity="10.0"/> <!-- Tag to limit torque and velocity within gazebo sim to make movement feel smooth-->
@@ -62,5 +63,5 @@
         <visual>
             <geometry>
-                <cylinder radius = "0.05" length="0.04"/>
+                <cylinder radius = "0.0691" length="0.065"/>
             </geometry>
             <material name = "blue"/>
@@ -68,9 +69,9 @@
         <collision>
             <geometry>
-                <sphere radius = "0.05"/>
+                <sphere radius = "0.0691"/>
             </geometry>
         </collision>
-        <xacro:inertial_cylinder mass = "0.1" length = "0.04" radius = "0.05">
-            <origin xyz = "0 0 0" rpy = "0 0 0"/>
+        <xacro:inertial_cylinder mass="0.1" length="0.065" radius="0.0691">
+            <origin xyz="0 0 0" rpy="0 0 0"/>
         </xacro:inertial_cylinder>
     </link>
@@ -79,5 +80,5 @@
         <parent link = "base_link"/>
         <child link = "right_wheel_link"/>
-        <origin xyz = "0 -0.175 0" rpy = "${pi/2} 0 0"/>
+        <origin xyz = "0 -0.255 0" rpy = "${pi/2} 0 0"/>
         <axis xyz = "0 0 -1"/>
         <limit effort="0.05" velocity="10.0"/> <!-- Tag to limit torque and velocity within gazebo sim to make movement feel smooth-->
@@ -86,5 +87,5 @@
         <visual>
             <geometry>
-                <cylinder radius = "0.05" length="0.04"/>
+                <cylinder radius = "0.0691" length="0.065"/>
             </geometry>
             <material name = "blue"/>
@@ -92,9 +93,9 @@
         <collision>
             <geometry>
-                <sphere radius = "0.05"/>
+                <sphere radius = "0.0691"/>
             </geometry>
         </collision>
-        <xacro:inertial_cylinder mass = "0.1" length = "0.04" radius = "0.05">
-            <origin xyz = "0 0 0" rpy = "0 0 0"/>
+        <xacro:inertial_cylinder mass="0.1" length="0.065" radius="0.0691">
+            <origin xyz="0 0 0" rpy="0 0 0"/>
         </xacro:inertial_cylinder>
     </link>
@@ -103,21 +104,41 @@
         <parent link = "chassis_link" />
         <child link = "caster_wheel_link"/>
-        <origin xyz = "0.24 0 0"/>
+        <origin xyz = "0 0 -0.035"/>
     </joint>
     <link name ="caster_wheel_link">
         <visual>
             <geometry>
-                <sphere radius = "0.05"/>
+                <sphere radius = "0.0691"/>
+            </geometry>
+            <material name = "white"/>
+        </visual>
+        <collision>
+            <geometry>
+                <sphere radius = "0.0691"/>
+            </geometry>
+        </collision>
+        <xacro:inertial_sphere mass="0.1" radius="0.0691">
+            <origin xyz="0 0 0" rpy="0 0 0"/>
+        </xacro:inertial_sphere>
+    </link>
+    <!-- BALL COLLECTION MECHANISM LINK -->
+    <joint name = "ball_collection_mechanism_joint" type = "fixed">
+        <parent link = "chassis_link" />
+        <child link = "ball_collection_mechanism_link"/>
+        <origin xyz = "0.580 0 -0.02"/>
+    </joint>
+    <link name ="ball_collection_mechanism_link">
+        <visual>
+            <geometry>
+                <box size = "0.12 0.21 0.1"/>
             </geometry>
             <material name = "black"/>
         </visual>
         <collision>
+            <origin xyz = "0 0 0"/>
             <geometry>
-                <sphere radius = "0.05"/>
+                <box size = "0.12 0.21 0.1"/>
             </geometry>
         </collision>
-        <xacro:inertial_sphere mass = "0.1" radius = "0.05">
-            <origin xyz = "0 0 0" rpy = "0 0 0"/>
-        </xacro:inertial_sphere>
     </link>
     <!-- Gazebo tag to make the caster wheel frictionless-->
